File: Digital_Remote.kicad_sch (KiCad schematic)
At the start: 56 parts, among them J1 Conn_01x11, J2 Conn_01x07, Q1 AO3401A, Q2 Q_NPN_BEC, SW1 SW_SPDT, U1 STM32F103C8Tx, U2 MP1584, U3 AMS1117-3.3, U4 MPU-6050, U5 AS01-SPI, Y1 8Mhz, Y2 32KHz

Commit message: Change schematic
Parts:
- removed BT1: 3V, symbol Device:Battery_Cell
- removed C2, C6: 20p, Capacitor_SMD:C_0603_1608Metric, symbol Device:C_Small
- removed J1: Conn_01x11, symbol Connector_Generic:Conn_01x11
- removed J2: Conn_01x07, symbol Connector_Generic:Conn_01x07
- removed Y2: 32KHz, Crystal:Crystal_SMD_3215-2Pin_3.2x1.5mm, symbol Device:Crystal_Small
- added D4: S7, Diode_SMD:D_SOD-123, symbol Device:D_Schottky_Small
- added J1, J10, J11, J12, J2, J5, J6, J7, J8, J9: Conn_01x03, MyConnector:con_01x03_W2.5mm-H2.5mm, symbol Connector_Generic:Conn_01x03
- added J13, J14: Conn_01x04, MyConnector:con_01x04_W2.5mm-H2.5mm, symbol Connector_Generic:Conn_01x04
- added J15: USB_C_Receptacle_USB2.0, Connector_USB:USB_C_Receptacle_XKB_U262-16XN-4BVC11, symbol Connector:USB_C_Receptacle_USB2.0
- added J16: Conn_01x02, Connector_PinHeader_2.54mm:PinHeader_1x02_P2.54mm_Vertical, symbol Connector_Generic:Conn_01x02
- added R16: 10k, Resistor_SMD:R_0603_1608Metric, symbol Device:R_Small
- added SW2: BIND, Button_Switch_THT:SW_PUSH_6mm_H5mm, symbol Switch:SW_Push
- BZ1: footprint (none) -> Buzzer_Beeper:Buzzer_12x9.5RM7.6
- D1: footprint (none) -> Diode_SMD:D_SMA
- D2: footprint (none) -> Diode_SMD:D_SOD-123
- J3, J4: renamed from J?; footprint (none) -> MyConnector:con_01x04_W2.5mm-H2.5mm
- Q2: footprint (none) -> Package_TO_SOT_SMD:SOT-23
- SW1: footprint (none) -> Button_Switch_THT:SW_CuK_JS202011CQN_DPDT_Straight
- U2: footprint (none) -> Package_SO:SOIC-8-1EP_3.9x4.9mm_P1.27mm_EP2.41x3.81mm
- U5: footprint myCustomLibs:AS01-SPI -> Wireless:AS01-SPIPX-NRF24
Connections:
- net B+ is gone; now on net VCC: R11.1
- net VBAT is gone; now on net +3V3: U1.1 (VBAT)
- net +3V3: now also J1.2 (Pin_2), J10.2 (Pin_2), J11.2 (Pin_2), J12.2 (Pin_2), J13.2 (Pin_2), J14.2 (Pin_2), J2.2 (Pin_2), J5.2 (Pin_2), J6.2 (Pin_2), J7.2 (Pin_2), J8.2 (Pin_2), J9.2 (Pin_2), SW2.2
- net +5V: now also D4.1 (K)
- net AUX_1: now also J1.3 (Pin_3)
- net AUX_2: now also J9.3 (Pin_3)
- net AUX_3: now also J10.3 (Pin_3)
- net AUX_4: now also J11.3 (Pin_3)
- net AUX_5: now also J12.3 (Pin_3)
- net BTN_BIND: now also R16.1, SW2.1
- net GND: now also J1.1 (Pin_1), J10.1 (Pin_1), J11.1 (Pin_1), J12.1 (Pin_1), J13.1 (Pin_1), J14.1 (Pin_1), J15.A1 (GND), J15.A12 (GND), J15.B1 (GND), J15.B12 (GND), J15.S1 (SHIELD), J16.1 (Pin_1), J2.1 (Pin_1), J5.1 (Pin_1), J6.1 (Pin_1), J7.1 (Pin_1), J8.1 (Pin_1), J9.1 (Pin_1), R16.2
- net J1_X: now also J13.4 (Pin_4)
- net J1_Y: now also J13.3 (Pin_3)
- net J2_X: now also J14.4 (Pin_4)
- net J2_Y: now also J14.3 (Pin_3)
- net NRF_CE: now also U1.29 (PA8); no longer U1.30 (PA9)
- net NRF_CSN: now also U1.30 (PA9); no longer U1.29 (PA8)
- net SWA: now also J5.3 (Pin_3)
- net SWB: now also J6.3 (Pin_3)
- net SWC: now also J7.3 (Pin_3)
- net SWD: now also J8.3 (Pin_3)
- net SWE: now also J2.3 (Pin_3)
- net VCC: now also J16.2 (Pin_2)
- net USB_D-: now reaches U1.32 (PA11)
- net USB_D-: now also J15.A7 (D-), J15.B7 (D-)
- net USB_D+: now reaches U1.33 (PA12)
- net USB_D+: now also J15.A6 (D+), J15.B6 (D+)
- net LSE_IN: no longer names the net of U1.3 (PC14)
- net LSE_OUT: no longer names the net of U1.4 (PC15)
- new net VBUS: D4.2 (A), J15.A4 (VBUS), J15.A9 (VBUS), J15.B4 (VBUS), J15.B9 (VBUS)
- no-connect marks 8 -> 13
Other:
- moved on the sheet: C11, C13, C14, C15, C7, D1, D3, J3, J4, L2, Q1, R14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
